File: hardware/devhub/relays.kicad_sch (KiCad schematic)
At the start: 17 parts, among them J5 Banana COM 1, J6 Banana NC 1, J7 Banana COM 2, J8 Banana NC 2, K1 G5Q-1 DC5, K2 G5Q-1 DC5, SW1 relè on/off, SW2 relè on/off, U9 ULN2003A

Commit message: Review 02, R02-06: ULN2003V12 relay driver, three channels in parallel per relay (D33)
Parts:
- U9: value ULN2003A -> ULN2003V12
Connections:
- net RLY1: now also U9.2 (I2), U9.3 (I3)
- net RLY1_COIL: now also U9.14 (O3), U9.15 (O2)
- net RLY2: now also U9.4 (I4), U9.5 (I5), U9.6 (I6); no longer U9.2 (I2)
- net RLY2_COIL: now also U9.11 (O6), U9.12 (O5), U9.13 (O4); no longer U9.15 (O2)
- no-connect marks 10 -> 2
Other:
- note added: "Bobina G5Q-1 senza polarità: pin 5 a +5V, pin 1 a tre uscite in parallelo del ULN2003V12 (diodi di ricircolo nel driver, COM a +5V)."
- note removed: "Bobina G5Q-1 senza polarità: pin 5 a +5V, pin 1 al ULN2003 (diodi di ricircolo nel ULN, COM a +5V)."
Changed lines of the file:
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@@
 		(company "devhub")
 	)
-	(text "Bobina G5Q-1 senza polarità: pin 5 a +5V, pin 1 al ULN2003 (diodi di ricircolo nel ULN, COM a +5V)."
+	(text "Bobina G5Q-1 senza polarità: pin 5 a +5V, pin 1 a tre uscite in parallelo del ULN2003V12 (diodi di ricircolo nel driver, COM a +5V)."
 		(exclude_from_sim no)
 		(at 10.16 152.4 0)
@@
 	)
 	(no_connect
-		(at 55.88 111.76)
-	)
-	(no_connect
-		(at 35.56 116.84)
-	)
-	(no_connect
-		(at 55.88 116.84)
-	)
-	(no_connect
-		(at 35.56 119.38)
-	)
-	(no_connect
-		(at 35.56 111.76)
-	)
-	(no_connect
 		(at 55.88 121.92)
-	)
-	(no_connect
-		(at 35.56 114.3)
 	)
 	(no_connect
 		(at 35.56 121.92)
 	)
-	(no_connect
-		(at 55.88 119.38)
-	)
-	(no_connect
-		(at 55.88 114.3)
-	)
-	(wire
-		(pts
-			(xy 55.88 109.22) (xy 187.96 109.22)
+	(wire
+		(pts
+			(xy 60.96 109.22) (xy 187.96 109.22)
 		)
 		(stroke
@@
 	(global_label "RLY1"
 		(shape bidirectional)
-		(at 35.56 106.68 180)
+		(at 30.48 106.68 180)
 		(fields_autoplaced yes)
 		(effects
@@
 		)
 		(property "Intersheetrefs" "${INTERSHEET_REFS}"
-			(at 35.56 106.68 0)
+			(at 30.48 106.68 0)
 			(hide yes)
 			(show_name no)
@@
 	(global_label "RLY2"
 		(shape bidirectional)
-		(at 35.56 109.22 180)
+		(at 30.48 114.3 180)
 		(fields_autoplaced yes)
 		(effects
@@
 		)
 		(property "Intersheetrefs" "${INTERSHEET_REFS}"
-			(at 35.56 109.22 0)
+			(at 30.48 114.3 0)
 			(hide yes)
 			(show_name no)
@@
 			)
 		)
-		(property "Value" "ULN2003A"
+		(property "Value" "ULN2003V12"
 			(at 38.1 96.52 0)
 			(show_name no)
@@
 			)
 		)
-		(property "Datasheet" "http://www.ti.com/lit/ds/symlink/uln2003a.pdf"
+		(property "Datasheet" "https://www.ti.com/lit/ds/symlink/uln2003v12.pdf"
 			(at 45.72 111.76 0)
 			(hide yes)
@@
 			)
 		)
-		(property "Description" "High Voltage, High Current Darlington Transistor Arrays, SOIC16/SOIC16W/DIP16/TSSOP16"
+		(property "Description" "7-channel low-side relay driver, NMOS outputs, clamp diodes to COM; pin-compatible with ULN2003A"
 			(at 45.72 111.76 0)
 			(hide yes)
@@
 		)
 	)
+	(wire
+		(pts
+			(xy 30.48 106.68) (xy 35.56 106.68)
+		)
+		(stroke
+			(width 0)
+			(type default)
+		)
+	)
+	(wire
+		(pts
+			(xy 33.02 109.22) (xy 35.56 109.22)
+		)
+		(stroke
+			(width 0)
+			(type default)
+		)
+	)
+	(wire
+		(pts
+			(xy 33.02 111.76) (xy 35.56 111.76)
+		)
+		(stroke
+			(width 0)
+			(type default)
+		)
+	)
+	(wire
+		(pts
+			(xy 33.02 106.68) (xy 33.02 111.76)
+		)
+		(stroke
+			(width 0)
+			(type default)
+		)
+	)
+	(junction
+		(at 33.02 106.68)
+		(diameter 0)
+		(color 0 0 0 0)
+	)
+	(junction
+		(at 33.02 109.22)
+		(diameter 0)
+		(color 0 0 0 0)
+	)
+	(wire
+		(pts
+			(xy 30.48 114.3) (xy 35.56 114.3)
+		)
+		(stroke
+			(width 0)
+			(type default)
+		)
+	)
+	(wire
+		(pts
+			(xy 33.02 116.84) (xy 35.56 116.84)
+		)
+		(stroke
+			(width 0)
+			(type default)
+		)
+	)
+	(wire
+		(pts
+			(xy 33.02 119.38) (xy 35.56 119.38)
+		)
+		(stroke
+			(width 0)
+			(type default)
+		)
+	)
+	(wire
+		(pts
+			(xy 33.02 114.3) (xy 33.02 119.38)
+		)
+		(stroke
+			(width 0)
+			(type default)
+		)
+	)
+	(junction
+		(at 33.02 114.3)
+		(diameter 0)
+		(color 0 0 0 0)
+	)
+	(junction
+		(at 33.02 116.84)
+		(diameter 0)
+		(color 0 0 0 0)
+	)
+	(wire
+		(pts
+			(xy 55.88 109.22) (xy 58.42 109.22)
+		)
+		(stroke
+			(width 0)
+			(type default)
+		)
+	)
+	(wire
+		(pts
+			(xy 55.88 111.76) (xy 58.42 111.76)
+		)
+		(stroke
+			(width 0)
+			(type default)
+		)
+	)
+	(wire
+		(pts
+			(xy 58.42 106.68) (xy 58.42 111.76)
+		)
+		(stroke
+			(width 0)
+			(type default)
+		)
+	)
+	(junction
+		(at 58.42 106.68)
+		(diameter 0)
+		(color 0 0 0 0)
+	)
+	(junction
+		(at 58.42 109.22)
+		(diameter 0)
+		(color 0 0 0 0)
+	)
+	(wire
+		(pts
+			(xy 55.88 114.3) (xy 60.96 114.3)
+		)
+		(stroke
+			(width 0)
+			(type default)
+		)
+	)
+	(wire
+		(pts
+			(xy 55.88 116.84) (xy 60.96 116.84)
+		)
+		(stroke
+			(width 0)
+			(type default)
+		)
+	)
+	(wire
+		(pts
+			(xy 55.88 119.38) (xy 60.96 119.38)
+		)
+		(stroke
+			(width 0)
+			(type default)
+		)
+	)
+	(wire
+		(pts
+			(xy 60.96 109.22) (xy 60.96 119.38)
+		)
+		(stroke
+			(width 0)
+			(type default)
+		)
+	)
+	(junction
+		(at 60.96 114.3)
+		(diameter 0)
+		(color 0 0 0 0)
+	)
+	(junction
+		(at 60.96 116.84)
+		(diameter 0)
+		(color 0 0 0 0)
+	)
 	(symbol
