File: hardware/devhub/port_a.kicad_sch (KiCad schematic)
At the start: 18 parts, among them J501 USB-A, Q501 AO3400A, SW501 porta on/off, U501 PI3USB4002A

Commit message: Review 02, R02-01: remove USBLC6 from downstream ports (D27)
Adds the electrical review 02 document.

The USBLC6 VBUS pin sat on the switched port VBUS: its internal diodes fed
current from the data lines into the supply (an "off" port at ~2.6 V with a
self-powered board) and routed data overvoltage to 5 V, bypassing the 24 V
tolerance of the PI3USB4002A. Downstream ESD protection is now the one
integrated in the switch (10 kV IEC); the upstream port keeps its USBLC6.

Connectivity checked, ERC clean.
Parts:
- removed D501: USBLC6-2SC6, Package_TO_SOT_SMD:SOT-23-6, symbol Power_Protection:USBLC6-2SC6
Connections:
- net DM_SW is gone; now on net DM_C: U501.7 (C0-)
- net DP_SW is gone; now on net DP_C: U501.8 (C0+)
Changed lines of the file:
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@@
 	(wire
 		(pts
-			(xy 86.36 71.12) (xy 111.76 71.12)
+			(xy 86.36 71.12) (xy 96.52 71.12)
 		)
 		(stroke
@@
 	(wire
 		(pts
-			(xy 116.84 66.04) (xy 116.84 63.5)
+			(xy 96.52 139.7) (xy 101.6 139.7)
 		)
 		(stroke
@@
 	(wire
 		(pts
-			(xy 96.52 139.7) (xy 101.6 139.7)
+			(xy 160.02 142.24) (xy 179.07 142.24)
 		)
 		(stroke
@@
 	(wire
 		(pts
-			(xy 160.02 142.24) (xy 179.07 142.24)
+			(xy 40.64 78.74) (xy 66.04 78.74)
 		)
 		(stroke
@@
 	(wire
 		(pts
-			(xy 40.64 78.74) (xy 66.04 78.74)
+			(xy 86.36 73.66) (xy 96.52 73.66)
 		)
 		(stroke
 			(width 0)
 			(type default)
-		)
-	)
-	(wire
-		(pts
-			(xy 86.36 73.66) (xy 111.76 73.66)
-		)
-		(stroke
-			(width 0)
-			(type default)
-		)
-	)
-	(label "VBUS"
-		(at 116.84 63.5 90)
-		(effects
-			(font
-				(size 1.27 1.27)
-			)
-			(justify left bottom)
 		)
 	)
@@
 		)
 	)
-	(label "DM_C"
-		(at 121.92 73.66 0)
-		(effects
-			(font
-				(size 1.27 1.27)
-			)
-			(justify left bottom)
-		)
-	)
 	(label "DIS_D"
 		(at 101.6 139.7 0)
@@
 		)
 	)
-	(label "DP_C"
-		(at 121.92 71.12 0)
-		(effects
-			(font
-				(size 1.27 1.27)
-			)
-			(justify left bottom)
-		)
-	)
 	(label "LED2_K"
 		(at 160.02 142.24 0)
@@
 		)
 	)
-	(label "DM_SW"
-		(at 93.98 73.66 0)
+	(label "DM_C"
+		(at 96.52 73.66 0)
 		(effects
 			(font
@@
 		)
 	)
-	(label "DP_SW"
-		(at 93.98 71.12 0)
+	(label "DP_C"
+		(at 96.52 71.12 0)
 		(effects
 			(font
@@
 	)
 	(symbol
-		(lib_id "Power_Protection:USBLC6-2SC6")
-		(at 116.84 71.12 0)
-		(unit 1)
-		(body_style 1)
-		(exclude_from_sim no)
-		(in_bom yes)
-		(on_board yes)
-		(in_pos_files yes)
-		(dnp no)
-		(property "Reference" "D501"
-			(at 120.65 63.5 0)
-			(show_name no)
-			(do_not_autoplace no)
-			(effects
-				(font
-					(size 1.27 1.27)
-				)
-				(justify left)
-			)
-		)
-		(property "Value" "USBLC6-2SC6"
-			(at 120.65 60.96 0)
-			(show_name no)
-			(do_not_autoplace no)
-			(effects
-				(font
-					(size 1.27 1.27)
-				)
-				(justify left)
-			)
-		)
-		(property "Footprint" "Package_TO_SOT_SMD:SOT-23-6"
-			(at 116.84 71.12 0)
-			(hide yes)
-			(show_name no)
-			(do_not_autoplace no)
-			(effects
-				(font
-					(size 1.27 1.27)
-				)
-			)
-		)
-		(property "Datasheet" "https://www.st.com/resource/en/datasheet/usblc6-2.pdf"
-			(at 116.84 71.12 0)
-			(hide yes)
-			(show_name no)
-			(do_not_autoplace no)
-			(effects
-				(font
-					(size 1.27 1.27)
-				)
-			)
-		)
-		(property "Description" "Very low capacitance ESD protection diode, 2 data-line, SOT-23-6"
-			(at 116.84 71.12 0)
-			(hide yes)
-			(show_name no)
-			(do_not_autoplace no)
-			(effects
-				(font
-					(size 1.27 1.27)
-				)
-			)
-		)
-		(pin "1"
-		)
-		(pin "2"
-		)
-		(pin "3"
-		)
-		(pin "4"
-		)
-		(pin "5"
-		)
-		(pin "6"
-		)
-		(instances
-			(project "devhub"
-				(path "/af6ea7d8-d1ba-5fc6-aec8-abf514847630/0c5617cc-af51-5b03-9838-7bc06ac23dd1"
-					(reference "D501")
-					(unit 1)
-				)
-			)
-		)
-	)
-	(symbol
 		(lib_id "Transistor_FET:AO3400A")
 		(at 93.98 144.78 0)
@@
 					(unit 1)
 				)
-			)
-		)
-	)
-	(symbol
-		(lib_id "power:GND")
-		(at 116.84 78.74 0)
-		(unit 1)
-		(body_style 1)
-		(exclude_from_sim no)
-		(in_bom yes)
-		(on_board yes)
-		(in_pos_files yes)
-		(dnp no)
-		(property "Reference" "#PWR5007"
-			(at 116.84 78.74 0)
-			(hide yes)
-			(show_name no)
-			(do_not_autoplace no)
-			(effects
-				(font
-					(size 1.27 1.27)
-				)
-			)
-		)
-		(property "Value" "GND"
-			(at 116.84 83.14 0)
-			(show_name no)
-			(do_not_autoplace no)
-			(effects
-				(font
-					(size 1.27 1.27)
-				)
-			)
-		)
-		(property "Footprint" ""
-			(at 116.84 78.74 0)
-			(hide yes)
-			(show_name no)
-			(do_not_autoplace no)
-			(effects
-				(font
-					(size 1.27 1.27)
-				)
-			)
-		)
-		(property "Datasheet" ""
-			(at 116.84 78.74 0)
-			(hide yes)
-			(show_name no)
-			(do_not_autoplace no)
-			(effects
-				(font
-					(size 1.27 1.27)
-				)
-			)
-		)
-		(property "Description" ""
-			(at 116.84 78.74 0)
-			(hide yes)
-			(show_name no)
-			(do_not_autoplace no)
-			(effects
-				(font
-					(size 1.27 1.27)
-				)
-			)
-		)
-		(pin "1"
-		)
-		(instances
-			(project "devhub"
-				(path "/af6ea7d8-d1ba-5fc6-aec8-abf514847630/0c5617cc-af51-5b03-9838-7bc06ac23dd1"
-					(reference "#PWR5007")
-					(unit 1)
-				)

Commit message: Intial PCB layout
Parts:
- SW501: footprint Button_Switch_THT:SW_PUSH_6mm_H13mm -> Button_Switch_SMD:SW_SPST_PTS645Sx43SMTR92
- U501: footprint (none) -> lcsc_footprints:C3657361_UQFN-10_L2_0-W1_5-P0_50-TL
Changed lines of the file:
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@@
 			)
 		)
-		(property "Footprint" ""
+		(property "Footprint" "lcsc_footprints:C3657361_UQFN-10_L2_0-W1_5-P0_50-TL"
 			(at 76.2 76.2 0)
 			(hide yes)
@@
 			)
 		)
-		(property "Footprint" "Button_Switch_THT:SW_PUSH_6mm_H13mm"
+		(property "Footprint" "Button_Switch_SMD:SW_SPST_PTS645Sx43SMTR92"
 			(at 182.88 157.48 0)
 			(hide yes)

Commit message: PCB rules in KiCad, USB pair names, eFuse output bypass and U2 thermal vias (D44-D50)
Stackup JLC04161H-7628, netclasses and custom DRC rules (devhub.kicad_dru) from
docs/regole-pcb.md, with a section for the checks that DRC cannot cover. C7 1 uF on
the TPS259470A output before the shunt (D48). USB nets renamed to DP/DN so KiCad
recognizes the differential pairs (D49). U2 footprint with 0.3 mm thermal vias, open
on both sides for the prototype; encroached vias and a JLCPCB order note for
production (D50). Also includes stock part codes, cost comparison and placement rules
(D44-D47).
Parts:
- C501, C503, C504: digikey (none) -> 1276-1000-1-ND; lcsc (none) -> C1591; mouser (none) -> 187-CL10B104KB8NNNC; warehouse (none) -> 235
- C502: digikey (none) -> 490-GRM21BZ71A226ME15LCT-ND; lcsc (none) -> C907991; mouser (none) -> 81-GRM21BZ71A226ME5L; warehouse (none) -> 300
- C505: footprint Capacitor_SMD:CP_Elec_6.3x7.7 -> Capacitor_SMD:CP_Elec_6.3x5.8; digikey (none) -> PCE3783CT-ND; lcsc (none) -> C128532; mouser (none) -> 667-EEE-FK1C101P; warehouse (none) -> 184
- C506: footprint Capacitor_SMD:C_0805_2012Metric -> Capacitor_SMD:C_0603_1608Metric; digikey (none) -> 1276-1184-1-ND; lcsc (none) -> C29936; mouser (none) -> 187-CL10B105KA8NNNC; warehouse (none) -> 240
- D502: digikey (none) -> 160-1423-1-ND; lcsc (none) -> C913075; mouser (none) -> 859-LTST-C171GKT
- D503: digikey (none) -> 160-1427-1-ND; lcsc (none) -> C284871; mouser (none) -> 859-LTST-C171KRKT
- J501: digikey (none) -> 2092-KUSBX-AS1N-B-ND; lcsc (none) -> C7212838; mouser (none) -> 806-KUSBX-AS1N-B
- Q501: digikey (none) -> 785-1000-1-ND; lcsc (none) -> C20917; mouser (none) -> 621-DMN3404L-7
- R501: digikey (none) -> 311-100FRCT-ND; lcsc (none) -> C137392; mouser (none) -> 603-RC1206FR-07100RL
- R504, R505: digikey (none) -> 311-100KHRCT-ND; lcsc (none) -> C2906980; mouser (none) -> 603-RC0603FR-07100KL; warehouse (none) -> 247
- R506, R507: digikey (none) -> 311-1.00KHRCT-ND; lcsc (none) -> C21190; mouser (none) -> 603-RC0603FR-071KL; warehouse (none) -> 284
- SW501: digikey (none) -> CKN10820CT-ND; lcsc (none) -> C285485; mouser (none) -> 611-645SL70SMTR92LFS
- U501: digikey (none) -> 31-PI3USB4002AZUAEXCT-ND; lcsc (none) -> C6735706; mouser (none) -> 621-PI3USB4002A
Connections:
- net DM_C renamed CONN_DN
- net DP_C renamed CONN_DP
- net HUB_DM renamed HUB_DN
