File: hardware/devhub/devhub.kicad_sch (KiCad schematic)
At the start: 0 parts

Commit message: Schematic: keep only host system LED, merge VBUS switches into hub sheet (D82, D83)
- remove relay LED (D90/R90) and power LED (D92/R92)
- move UCS2114 VBUS switches into the hub sheet, renamed to
  "Hub USB e switch VBUS"
- move the host LED into the MCU sheet as a local net
- drop the switches and ui sheets; update netclass patterns and docs
Other:
- sheet Hub USB2517 renamed Hub USB e switch VBUS
- removed sheet LED di stato
- removed sheet Switch VBUS porte
Changed lines of the file:
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@@
+	)
+	(sheet
+		(at 15.24 91.44)
+		(size 76.2 20.32)
+		(exclude_from_sim no)
+		(in_bom yes)
+		(on_board yes)
+		(dnp no)
+		(fields_autoplaced yes)
+		(stroke
+			(width 0.1524)
+			(type solid)
+		)
+		(fill
+			(color 0 0 0 0)
+		)
+		(property "Sheetname" "MCU STM32G0B1"
+			(at 15.24 90.74 0)
+			(show_name no)
+			(do_not_autoplace no)
+			(effects
+				(font
+					(size 1.27 1.27)
+				)
+				(justify left bottom)
+			)
+		)
+		(property "Sheetfile" "mcu.kicad_sch"
+			(at 15.24 112.36 0)
+			(show_name no)
+			(do_not_autoplace no)
+			(effects
+				(font
+					(size 1.27 1.27)
+				)
+				(justify left top)
+			)
+		)
+		(instances
+			(project "devhub"
+				(path "/af6ea7d8-d1ba-5fc6-aec8-abf514847630"
+					(page "4")
+				)
+			)
+		)
 	)
 	(sheet
@@
 			(color 0 0 0 0)
 		)
-		(property "Sheetname" "Switch VBUS porte"
+		(property "Sheetname" "Relè ausiliario"
 			(at 15.24 121.22 0)
 			(show_name no)
@@
 			)
 		)
-		(property "Sheetfile" "switches.kicad_sch"
+		(property "Sheetfile" "relays.kicad_sch"
 			(at 15.24 142.84 0)
 			(show_name no)
@@
 				(path "/af6ea7d8-d1ba-5fc6-aec8-abf514847630"
 					(page "5")
-				)
-			)
-		)
-	)
-	(sheet
-		(at 15.24 91.44)
-		(size 76.2 20.32)
-		(exclude_from_sim no)
-		(in_bom yes)
-		(on_board yes)
-		(dnp no)
-		(fields_autoplaced yes)
-		(stroke
-			(width 0.1524)
-			(type solid)
-		)
-		(fill
-			(color 0 0 0 0)
-		)
-		(property "Sheetname" "MCU STM32G0B1"
-			(at 15.24 90.74 0)
-			(show_name no)
-			(do_not_autoplace no)
-			(effects
-				(font
-					(size 1.27 1.27)
-				)
-				(justify left bottom)
-			)
-		)
-		(property "Sheetfile" "mcu.kicad_sch"
-			(at 15.24 112.36 0)
-			(show_name no)
-			(do_not_autoplace no)
-			(effects
-				(font
-					(size 1.27 1.27)
-				)
-				(justify left top)
-			)
-		)
-		(instances
-			(project "devhub"
-				(path "/af6ea7d8-d1ba-5fc6-aec8-abf514847630"
-					(page "4")
-				)
-			)
-		)
-	)
-	(sheet
-		(at 15.24 152.4)
-		(size 76.2 20.32)
-		(exclude_from_sim no)
-		(in_bom yes)
-		(on_board yes)
-		(dnp no)
-		(fields_autoplaced yes)
-		(stroke
-			(width 0.1524)
-			(type solid)
-		)
-		(fill
-			(color 0 0 0 0)
-		)
-		(property "Sheetname" "Relè ausiliario"
-			(at 15.24 151.7 0)
-			(show_name no)
-			(do_not_autoplace no)
-			(effects
-				(font
-					(size 1.27 1.27)
-				)
-				(justify left bottom)
-			)
-		)
-		(property "Sheetfile" "relays.kicad_sch"
-			(at 15.24 173.32 0)
-			(show_name no)
-			(do_not_autoplace no)
-			(effects
-				(font
-					(size 1.27 1.27)
-				)
-				(justify left top)
-			)
-		)
-		(instances
-			(project "devhub"
-				(path "/af6ea7d8-d1ba-5fc6-aec8-abf514847630"
-					(page "6")
 				)
 			)
@@
 			(project "devhub"
 				(path "/af6ea7d8-d1ba-5fc6-aec8-abf514847630"
-					(page "8")
+					(page "6")
 				)
 			)
@@
 			(project "devhub"
 				(path "/af6ea7d8-d1ba-5fc6-aec8-abf514847630"
-					(page "11")
+					(page "9")
 				)
 			)
@@
 			(color 0 0 0 0)
 		)
-		(property "Sheetname" "Hub USB2517"
+		(property "Sheetname" "Hub USB e switch VBUS"
 			(at 15.24 60.26 0)
 			(show_name no)
@@
 			(project "devhub"
 				(path "/af6ea7d8-d1ba-5fc6-aec8-abf514847630"
-					(page "9")
-				)
-			)
-		)
-	)
-	(sheet
-		(at 15.24 182.88)
-		(size 76.2 20.32)
-		(exclude_from_sim no)
-		(in_bom yes)
-		(on_board yes)
-		(dnp no)
-		(fields_autoplaced yes)
-		(stroke
-			(width 0.1524)
-			(type solid)
-		)
-		(fill
-			(color 0 0 0 0)
-		)
-		(property "Sheetname" "LED di stato"
-			(at 15.24 182.18 0)
-			(show_name no)
-			(do_not_autoplace no)
-			(effects
-				(font
-					(size 1.27 1.27)
-				)
-				(justify left bottom)
-			)
-		)
-		(property "Sheetfile" "ui.kicad_sch"
-			(at 15.24 203.8 0)
-			(show_name no)
-			(do_not_autoplace no)
-			(effects
-				(font
-					(size 1.27 1.27)
-				)
-				(justify left top)
-			)
-		)
-		(instances
-			(project "devhub"
-				(path "/af6ea7d8-d1ba-5fc6-aec8-abf514847630"
 					(page "7")
 				)
@@
 			(project "devhub"
 				(path "/af6ea7d8-d1ba-5fc6-aec8-abf514847630"
-					(page "10")
-				)
-			)
+					(page "8")
+				)
+			)
