File: hardware/devhub/mcu.kicad_sch (KiCad schematic)
At the start: 17 parts, among them J4 SWD, J9 UART debug, U3 STM32G0B1RET6

Commit message: Schematic v0.3: apply simplified requirements (D79-D81)
Update the existing KiCad project instead of starting over:
- MCU U3 replaced with STM32G0B1CEU6 (UFQFPN48) on the 48-pin pinout
- switches sheet: two UCS2114-1-V/LX on separate I2C buses replace
  TPS2561A, INA3221 and current shunts
- ports: single MCU-driven LED, discrete VBUS discharge removed
- remove USB-A port, spare hub header, second relay channel,
  input CC ADC filters and input shunt
- add UCS2114 symbol and footprint (Microchip land pattern C04-2421)
- align pinout, decisions, architecture and component docs
Parts:
- removed R46: 100k, Resistor_SMD:R_0603_1608Metric, symbol Device:R
- removed R47: 10k, Resistor_SMD:R_0603_1608Metric, symbol Device:R
- added R50, R51: 4.7k, Resistor_SMD:R_0603_1608Metric, symbol Device:R
- R42, R43, R44, R45: value 100k -> 10k; digikey 311-100KHRCT-ND -> 311-10.0KHRCT-ND; lcsc C2906980 -> C2906982; mouser 603-RC0603FR-07100KL -> 603-RC0603FR-0710KL; warehouse 247 -> 248
- U3: value STM32G0B1RET6 -> STM32G0B1CEU6; footprint Package_QFP:LQFP-64_10x10mm_P0.5mm -> Package_DFN_QFN:QFN-48-1EP_7x7mm_P0.5mm_EP5.6x5.6mm; symbol MCU_ST_STM32G0:STM32G0B1RETx -> MCU_ST_STM32G0:STM32G0B1CEUx; digikey 497-STM32G0B1RET6-ND -> 497-STM32G0B1CEU6-ND; lcsc C2829307 -> (none); mouser 511-STM32G0B1RET6 -> (none)
Connections:
- net BTN_P5 is gone; now on net NRST: U3.10 (PF2)
- net BTN_RLY2 is gone; now on net USB_MCU_DN: U3.33 (PA9/PA11)
- net DIS_P1 is gone; now on net FAULT_P4: U3.15 (PA4)
- net DIS_P5 is gone; now on net RLY1: U3.40 (PD2)
- net FAULT_P5 is gone; now on net FAULT_P2: U3.41 (PD3)
- net INA_ALERT is gone; now on net BTN_P2: U3.2 (PC14)
- net LED_FLT_P5 is gone; now on net SWDIO: U3.35 (PA13)
- net +3V3: now also U3.4 (VBAT), U3.5 (VREF+), R50.1, R51.1; no longer U3.7 (VREF+), U3.8 (VDD)
- net BTN_P1: now also U3.1 (PC13); no longer U3.3 (PC13)
- net BTN_P2: no longer U3.4 (PC14)
- net BTN_P3: now also U3.3 (PC15); no longer U3.5 (PC15)
- net BTN_P4: now also U3.24 (PB12); no longer U3.54 (PD4)
- net BTN_RLY1: now also U3.25 (PB13); no longer U3.32 (PB12)
- net EFUSE_FLT_N: now also U3.20 (PB1); no longer U3.28 (PB1)
- net EN_P1: now also U3.11 (PA0); no longer U3.13 (PC0)
- net EN_P2: now also U3.12 (PA1); no longer U3.25 (PC4)
- net EN_P3: now also U3.30 (PC6); no longer U3.48 (PC8)
- net EN_P4: now also U3.31 (PC7); no longer U3.24 (PA7)
- net FAULT_P1: now also U3.19 (PB0); no longer U3.16 (PC3)
- net FAULT_P2: no longer U3.39 (PC7)
- net FAULT_P3: now also U3.44 (PB5); no longer U3.1 (PC11)
- net FAULT_P4: no longer U3.53 (PD3)
- net GND: now also U3.49 (VSS), U3.7 (VSS); no longer U3.9 (VSS)
- net HUB_CFG_SEL2: now also U3.37 (PA15); no longer U3.47 (PA15)
- net HUB_RST_N: now also U3.9 (PF1); no longer U3.11 (PF1)
- net LED_HOST: now also U3.8 (PF0); no longer U3.36 (PA8)
- net NRST: no longer U3.12 (PF2)
- net OE_N_P1: now also U3.42 (PB3); no longer U3.14 (PC1)
- net OE_N_P2: now also U3.43 (PB4); no longer U3.26 (PC5)
- net OE_N_P3: now also U3.26 (PB14); no longer U3.49 (PC9)
- net OE_N_P4: now also U3.39 (PD1); no longer U3.51 (PD1)
- net RLY1: no longer U3.21 (PA4)
- net SWCLK: now also U3.36 (PA14); no longer U3.46 (PA14)
- net SWDIO: no longer U3.45 (PA13)
- net UART_RX: now also U3.14 (PA3); no longer U3.20 (PA3)
- net UART_TX: now also U3.13 (PA2); no longer U3.19 (PA2)
- net UCPD1_DBCC1: now also U3.29 (PA9/UCPD1_DBCC1); no longer U3.37 (PA9/UCPD1_DBCC1)
- net UCPD1_DBCC2: now also U3.32 (PA10/UCPD1_DBCC2); no longer U3.42 (PA10/UCPD1_DBCC2)
- net USB_MCU_DN: no longer U3.43 (PA9/PA11)
- net USB_MCU_DP: now also U3.34 (PA10/PA12); no longer U3.44 (PA10/PA12)
- net VBUS_DET: now also U3.21 (PB2); no longer U3.29 (PB2)
- net I2C2_SDA: now reaches U3.23 (PB11)
- net I2C2_SDA: now also R51.2
- net LED_P3: now reaches U3.27 (PB15)
- net CC1_ADC: no longer names the net of U3.17 (PA6)
- net CC2_ADC renamed LED_P2
- net DIS_P2: no longer names the net of U3.38 (PD0)
- removed net DIS_P3: U3.64 (PC10)
- removed net DIS_P4: U3.52 (PD2)
- removed net EN_P5: U3.55 (PD5)
- removed net LED_FLT_P1: U3.57 (PB3)
- removed net LED_FLT_P2: U3.58 (PB4)
- removed net LED_FLT_P3: U3.59 (PB5)
- removed net LED_FLT_P4: U3.50 (PD0)
- removed net OE_N_P5: U3.56 (PD6)
- net RLY2 renamed I2C2_SCL
- net I2C2_SCL: now also R50.2
- net SCL renamed I2C1_SCL
- net I2C1_SCL: now also U3.47 (PB8); no longer U3.62 (PB8)
- net SDA renamed I2C1_SDA
- net I2C1_SDA: now also U3.48 (PB9); no longer U3.63 (PB9)
- new net LED_P1: U3.16 (PA5)
- new net LED_P4: U3.28 (PA8)
- no-connect marks 10 -> 7
Other:
- note added: "Disaccoppiamento U3 (DS13560 fig. 15): C41 100 nF e C40 4,7 uF su VDD/VDDA (pin 6), C41 il più vicino; C42 100 nF su VREF+ (pin 5). VBAT (pin 4) collegato a VDD, senza condensatore. Pad esposto (pin 49) a GND."
- note added: "Pull-up 4,7 k: I2C1 (R40/R41) e I2C2 (R50/R51). Pull-up degli ALERT# nel foglio switches."
- note added: "R42-R45: pull-down 10 k sugli EN (PWR_EN degli UCS2114): VBUS spenta al reset e durante il bootloader."
- note added: "USB FS sulla porta 6 del hub (senza quarzo: HSI48 + CRS). I2C1: hub SMBus (0x2C) e UCS2114 U4 porte 1-2 (0x57); I2C2: UCS2114 U5 porte 3-4 (0x57). Per porta: EN (PWR_EN), OE_N (dati), FAULT (ALERT#), LED, BTN. Pinout in docs/pinout-mcu.md."
- note removed: "Disaccoppiamento U3 (DS13560 fig. 15): C41 100 nF e C40 4,7 uF sulla coppia VDD/VSS (pin 8/9), C41 il più vicino; C42 100 nF su VREF+ (pin 7). VBAT (pin 6) collegato a VDD, senza condensatore."
- note removed: "Pull-up: SCL/SDA 4,7 k; INA_ALERT 10 k (open-drain);"
- note removed: "R42-R46: pull-down sugli EN (porte spente al reset e durante il bootloader)."
- note removed: "USB FS sulla porta 6 del hub (senza quarzo: HSI48 + CRS). I2C1: INA3221 x2 (0x40, 0x41) e hub SMBus (0x2C). LED rossi e host dai GPIO (D38). Per porta: EN, OE_N, DIS, FAULT, BTN."
- title: MCU di controllo STM32G0B1RET6 -> MCU di controllo STM32G0B1CEU6

Commit message: Schematic: keep only host system LED, merge VBUS switches into hub sheet (D82, D83)
- remove relay LED (D90/R90) and power LED (D92/R92)
- move UCS2114 VBUS switches into the hub sheet, renamed to
  "Hub USB e switch VBUS"
- move the host LED into the MCU sheet as a local net
- drop the switches and ui sheets; update netclass patterns and docs
Parts:
- added D93: arancio, LED_SMD:LED_0805_2012Metric, symbol Device:LED
- added R93: 1k, Resistor_SMD:R_0603_1608Metric, symbol Device:R
Connections:
- net GND: now also D93.1 (K)
- net LED_HOST: now also R93.1
- new net LED_HOST_K: D93.2 (A), R93.2
Other:
- note added: "LED di sistema: solo host collegato (D93), acceso dal MCU (LED_HOST alto) a enumerazione completata (D82)."
- note added: "Pull-up 4,7 k: I2C1 (R40/R41) e I2C2 (R50/R51). Pull-up degli ALERT# nel foglio hub."
- note added: "host collegato"
- note removed: "Pull-up 4,7 k: I2C1 (R40/R41) e I2C2 (R50/R51). Pull-up degli ALERT# nel foglio switches."
- title: MCU di controllo STM32G0B1CEU6 -> MCU di controllo STM32G0B1CEU6 e LED host

Commit message: MCU 100 nF caps in 0402, U2/U3 fanout rule areas (D88)
- C41, C42, C46 to C_0402_1005Metric, warehouse ID 217 (CC0402KRX7R7BB104)
- Single U2_FANOUT and new U3_FANOUT rule areas for USB clearance exceptions
- Zone defaults: 1 mm corner radius, 0.1 mm min clearance
- Fix MCU pin numbers in D57 (UFQFPN48)
Parts:
- C41, C42, C46: footprint Capacitor_SMD:C_0603_1608Metric -> Capacitor_SMD:C_0402_1005Metric; digikey 1276-1000-1-ND -> 311-1338-1-ND; lcsc C1591 -> C60474; mouser 187-CL10B104KB8NNNC -> 603-CC402KRX7R7BB104; warehouse 235 -> 217
Changed lines of the file:
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@@
 			)
 		)
-		(property "Footprint" "Capacitor_SMD:C_0603_1608Metric"
+		(property "Footprint" "Capacitor_SMD:C_0402_1005Metric"
 			(at 128.27 127 0)
 			(hide yes)
@@
 			)
 		)
-		(property "warehouse" "235"
+		(property "warehouse" "217"
 			(at 128.27 127 0)
 			(hide yes)
@@
 			)
 		)
-		(property "lcsc" "C1591"
+		(property "lcsc" "C60474"
 			(at 128.27 127 0)
 			(hide yes)
@@
 			)
 		)
-		(property "mouser" "187-CL10B104KB8NNNC"
+		(property "mouser" "603-CC402KRX7R7BB104"
 			(at 128.27 127 0)
 			(hide yes)
@@
 			)
 		)
-		(property "digikey" "1276-1000-1-ND"
+		(property "digikey" "311-1338-1-ND"
 			(at 128.27 127 0)
 			(hide yes)
@@
 			)
 		)
-		(property "Footprint" "Capacitor_SMD:C_0603_1608Metric"
+		(property "Footprint" "Capacitor_SMD:C_0402_1005Metric"
 			(at 195.58 100.33 0)
 			(hide yes)
@@
 			)
 		)
-		(property "warehouse" "235"
+		(property "warehouse" "217"
 			(at 195.58 100.33 0)
 			(hide yes)
@@
 			)
 		)
-		(property "lcsc" "C1591"
+		(property "lcsc" "C60474"
 			(at 195.58 100.33 0)
 			(hide yes)
@@
 			)
 		)
-		(property "mouser" "187-CL10B104KB8NNNC"
+		(property "mouser" "603-CC402KRX7R7BB104"
 			(at 195.58 100.33 0)
 			(hide yes)
@@
 			)
 		)
-		(property "digikey" "1276-1000-1-ND"
+		(property "digikey" "311-1338-1-ND"
 			(at 195.58 100.33 0)
 			(hide yes)
@@
 			)
 		)
-		(property "Footprint" "Capacitor_SMD:C_0603_1608Metric"
+		(property "Footprint" "Capacitor_SMD:C_0402_1005Metric"
 			(at 152.4 116.84 0)
 			(hide yes)
@@
 			)
 		)
-		(property "warehouse" "235"
+		(property "warehouse" "217"
 			(at 152.4 116.84 0)
 			(hide yes)
@@
 			)
 		)
-		(property "lcsc" "C1591"
+		(property "lcsc" "C60474"
 			(at 152.4 116.84 0)
 			(hide yes)
@@
 			)
 		)
-		(property "mouser" "187-CL10B104KB8NNNC"
+		(property "mouser" "603-CC402KRX7R7BB104"
 			(at 152.4 116.84 0)
 			(hide yes)
@@
 			)
 		)
-		(property "digikey" "1276-1000-1-ND"
+		(property "digikey" "311-1338-1-ND"
 			(at 152.4 116.84 0)
 			(hide yes)
