File: hardware/devhub/port_c.kicad_sch (KiCad schematic)
At the start: 18 parts, among them J101 USB-C, Q101 AO3400A, SW101 porta on/off, U101 PI3USB4002A

Commit message: Intial PCB layout
Parts:
- SW101: footprint Button_Switch_THT:SW_PUSH_6mm_H13mm -> Button_Switch_SMD:SW_SPST_PTS645Sx43SMTR92
- U101: footprint (none) -> lcsc_footprints:C3657361_UQFN-10_L2_0-W1_5-P0_50-TL
Changed lines of the file:
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@@
 			)
 		)
-		(property "Footprint" "Button_Switch_THT:SW_PUSH_6mm_H13mm"
+		(property "Footprint" "Button_Switch_SMD:SW_SPST_PTS645Sx43SMTR92"
 			(at 182.88 157.48 0)
 			(hide yes)
@@
 			)
 		)
-		(property "Footprint" ""
+		(property "Footprint" "lcsc_footprints:C3657361_UQFN-10_L2_0-W1_5-P0_50-TL"
 			(at 76.2 76.2 0)
 			(hide yes)

Commit message: PCB rules in KiCad, USB pair names, eFuse output bypass and U2 thermal vias (D44-D50)
Stackup JLC04161H-7628, netclasses and custom DRC rules (devhub.kicad_dru) from
docs/regole-pcb.md, with a section for the checks that DRC cannot cover. C7 1 uF on
the TPS259470A output before the shunt (D48). USB nets renamed to DP/DN so KiCad
recognizes the differential pairs (D49). U2 footprint with 0.3 mm thermal vias, open
on both sides for the prototype; encroached vias and a JLCPCB order note for
production (D50). Also includes stock part codes, cost comparison and placement rules
(D44-D47).
Parts:
- C101, C103, C104: digikey (none) -> 1276-1000-1-ND; lcsc (none) -> C1591; mouser (none) -> 187-CL10B104KB8NNNC; warehouse (none) -> 235
- C102: digikey (none) -> 490-GRM21BZ71A226ME15LCT-ND; lcsc (none) -> C907991; mouser (none) -> 81-GRM21BZ71A226ME5L; warehouse (none) -> 300
- C106: footprint Capacitor_SMD:C_0805_2012Metric -> Capacitor_SMD:C_0603_1608Metric; digikey (none) -> 1276-1184-1-ND; lcsc (none) -> C29936; mouser (none) -> 187-CL10B105KA8NNNC; warehouse (none) -> 240
- D102: digikey (none) -> 160-1423-1-ND; lcsc (none) -> C913075; mouser (none) -> 859-LTST-C171GKT
- D103: digikey (none) -> 160-1427-1-ND; lcsc (none) -> C284871; mouser (none) -> 859-LTST-C171KRKT
- J101: digikey (none) -> 2073-USB4105-GF-ACT-ND; lcsc (none) -> C3020560; mouser (none) -> 640-USB4105-GF-A; warehouse (none) -> 279
- Q101: digikey (none) -> 785-1000-1-ND; lcsc (none) -> C20917; mouser (none) -> 621-DMN3404L-7
- R101: digikey (none) -> 311-100FRCT-ND; lcsc (none) -> C137392; mouser (none) -> 603-RC1206FR-07100RL
- R102, R103: digikey (none) -> 311-56KHRCT-ND; lcsc (none) -> C114630; mouser (none) -> 603-RC0603FR-0756KL
- R104, R105: digikey (none) -> 311-100KHRCT-ND; lcsc (none) -> C2906980; mouser (none) -> 603-RC0603FR-07100KL; warehouse (none) -> 247
- R106, R107: digikey (none) -> 311-1.00KHRCT-ND; lcsc (none) -> C21190; mouser (none) -> 603-RC0603FR-071KL; warehouse (none) -> 284
- SW101: digikey (none) -> CKN10820CT-ND; lcsc (none) -> C285485; mouser (none) -> 611-645SL70SMTR92LFS
- U101: digikey (none) -> 31-PI3USB4002AZUAEXCT-ND; lcsc (none) -> C6735706; mouser (none) -> 621-PI3USB4002A
Connections:
- net DM_C renamed CONN_DN
- net DP_C renamed CONN_DP
- net HUB_DM renamed HUB_DN

Commit message: Schematic v0.3: apply simplified requirements (D79-D81)
Update the existing KiCad project instead of starting over:
- MCU U3 replaced with STM32G0B1CEU6 (UFQFPN48) on the 48-pin pinout
- switches sheet: two UCS2114-1-V/LX on separate I2C buses replace
  TPS2561A, INA3221 and current shunts
- ports: single MCU-driven LED, discrete VBUS discharge removed
- remove USB-A port, spare hub header, second relay channel,
  input CC ADC filters and input shunt
- add UCS2114 symbol and footprint (Microchip land pattern C04-2421)
- align pinout, decisions, architecture and component docs
Parts:
- removed D103: rosso, LED_SMD:LED_0805_2012Metric, symbol Device:LED
- removed Q101: AO3400A, Package_TO_SOT_SMD:SOT-23, symbol Transistor_FET:AO3400A
- removed R101: 100 1206, Resistor_SMD:R_1206_3216Metric, symbol Device:R
- removed R105: 100k, Resistor_SMD:R_0603_1608Metric, symbol Device:R
- removed R107: 1k, Resistor_SMD:R_0603_1608Metric, symbol Device:R
Connections:
- net LED_PWR renamed LED
Other:
- note added: "LED: unico LED della porta, pilotato dal MCU: spento = disabilitata, acceso = abilitata, lampeggiante = guasto (D63)."
- note added: "VBUS dagli UCS2114 (foglio switches), con limite di corrente, blocco inverso e scarica automatica integrati. Dati: PI3USB4002A tra hub e connettore, OE_N (EN) alto = scollegato (pull-up: scollegato al reset); lato connettore tollera 24 V e si apre da solo sopra 4,75 V."
- note added: "la porta non lo impone: limite hw 2,5-2,9 A (UCS2114)"
- note removed: "DIS: scarica VBUS con Q1/R1 per ~100 ms dopo lo spegnimento."
- note removed: "VBUS dal load switch (foglio switches). Dati: PI3USB4002A tra hub e connettore, OE_N (EN) alto = scollegato (pull-up: scollegato al reset); lato connettore tollera 24 V e si apre da solo sopra 4,75 V."
- note removed: "la porta non lo impone: limite hw ~2,3 A"

Commit message: Schematic: keep only host system LED, merge VBUS switches into hub sheet (D82, D83)
- remove relay LED (D90/R90) and power LED (D92/R92)
- move UCS2114 VBUS switches into the hub sheet, renamed to
  "Hub USB e switch VBUS"
- move the host LED into the MCU sheet as a local net
- drop the switches and ui sheets; update netclass patterns and docs
Other:
- note added: "VBUS dagli UCS2114 (foglio hub), con limite di corrente, blocco inverso e scarica automatica integrati. Dati: PI3USB4002A tra hub e connettore, OE_N (EN) alto = scollegato (pull-up: scollegato al reset); lato connettore tollera 24 V e si apre da solo sopra 4,75 V."
- note removed: "VBUS dagli UCS2114 (foglio switches), con limite di corrente, blocco inverso e scarica automatica integrati. Dati: PI3USB4002A tra hub e connettore, OE_N (EN) alto = scollegato (pull-up: scollegato al reset); lato connettore tollera 24 V e si apre da solo sopra 4,75 V."
Changed lines of the file:
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@@
 		(company "devhub")
 	)
-	(text "VBUS dagli UCS2114 (foglio switches), con limite di corrente, blocco inverso e scarica automatica integrati. Dati: PI3USB4002A tra hub e connettore, OE_N (EN) alto = scollegato (pull-up: scollegato al reset); lato connettore tollera 24 V e si apre da solo sopra 4,75 V."
+	(text "VBUS dagli UCS2114 (foglio hub), con limite di corrente, blocco inverso e scarica automatica integrati. Dati: PI3USB4002A tra hub e connettore, OE_N (EN) alto = scollegato (pull-up: scollegato al reset); lato connettore tollera 24 V e si apre da solo sopra 4,75 V."
 		(exclude_from_sim no)
 		(at 10.16 16.51 0)

Commit message: PCB routing complete, package in values, MPN fields
- Routing finished; ESD_FANOUT rule area for D20 centre pins
- Vias keep inner-layer rings only where connected; GND reference vias
  next to SWD and I2C layer changes
- Value field of chip R/C/LED includes the package (0402...1206)
- New fields MPN lcsc, MPN mouser, MPN digikey; LCSC codes for R60/R61,
  U3, U4/U5 and supplier codes completed; JP2 marked DNP on the PCB
Parts:
- C101, C103, C104: value 100n -> 100n 0603; MPN digikey (none) -> CL10B104KB8NNNC; MPN lcsc (none) -> CL10B104KB8NNNC; MPN mouser (none) -> CL10B104KB8NNNC
- C102: value 22u 10V -> 22u 10V 0805; MPN digikey (none) -> GRM21BZ71A226ME15L; MPN lcsc (none) -> GRM21BZ71A226ME15L; MPN mouser (none) -> GRM21BZ71A226ME15L
- C106: value 1u 25V -> 1u 25V 0603; MPN digikey (none) -> CL10B105KA8NNNC; MPN lcsc (none) -> CL10B105KA8NNNC; MPN mouser (none) -> CL10B105KA8NNNC
- D102: value verde -> verde 0805; MPN digikey (none) -> LTST-C171GKT; MPN lcsc (none) -> LTST-C171GKT; MPN mouser (none) -> LTST-C171GKT
- J101: MPN digikey (none) -> USB4105-GF-A; MPN lcsc (none) -> USB4105-GF-A; MPN mouser (none) -> USB4105-GF-A
- R102, R103: value 56k -> 56k 0603; MPN digikey (none) -> RC0603FR-0756KL; MPN lcsc (none) -> RC0603FR-0756KL; MPN mouser (none) -> RC0603FR-0756KL
- R104: value 100k -> 100k 0603; MPN digikey (none) -> RC0603FR-07100KL; MPN lcsc (none) -> FRC0603F1003TS; MPN mouser (none) -> RC0603FR-07100KL
- R106: value 1k -> 1k 0603; MPN digikey (none) -> RC0603FR-071KL; MPN lcsc (none) -> 0603WAF1001T5E; MPN mouser (none) -> RC0603FR-071KL
- SW101: MPN digikey (none) -> PTS645SL70SMTR92 LFS; MPN lcsc (none) -> PTS645SL70SMTR92 LFS; MPN mouser (none) -> PTS645SL70SMTR92 LFS
- U101: MPN digikey (none) -> PI3USB4002AZUAEX; MPN lcsc (none) -> PI3USB4002AZUAEX; MPN mouser (none) -> PI3USB4002AZUAEX

Commit message: Test points, LED host moved, board finished (D92)
- 14 test points: GND loops TP1/TP10 (Keystone 5001), pads for +5V, +3V3,
  I2C1/I2C2, HUB_RST_N, EFUSE_FLT_N and VBUS_P1-P4
- D93/R93 moved to the rear, left of J1
- Button symbols: generic Value, function in Description; PCB aligned
- Docs: decision D92, components, PCB test rules, LED host position
Parts:
- SW101: value porta on/off -> Push button switch, generic, two pins
Changed lines of the file:
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@@
 			)
 		)
-		(property "Value" "porta on/off"
+		(property "Value" "Push button switch, generic, two pins"
 			(at 182.88 160.02 0)
 			(show_name no)
@@
 			)
 		)
-		(property "Description" "Push button switch, generic, two pins"
+		(property "Description" "porta on/off"
 			(at 182.88 157.48 0)
 			(hide yes)
